Commit message: Noetic port.

File: ros_ws/src/simulation/racer_description/urdf/racer_macros.xacro (robot description, xacro)
@@ -2,29 +2,29 @@
 <robot name="racer_macros" xmlns:xacro="http://www.ros.org/wiki/xacro">
   <!-- Inertias -->
-  <macro name="cylinder_inertia" params="m r h">
+  <xacro:macro name="cylinder_inertia" params="m r h">
     <inertia  ixx="${m*(3*r*r+h*h)/12}" ixy = "0" ixz = "0"
               iyy="${m*(3*r*r+h*h)/12}" iyz = "0"
               izz="${m*r*r/2}" />
-  </macro>
-  <macro name="box_inertia" params="m l b h">
+  </xacro:macro>
+  <xacro:macro name="box_inertia" params="m l b h">
     <inertia  ixx="${m*(b*b+h*h)/12}" ixy = "0" ixz = "0"
               iyy="${m*(l*l+h*h)/12}" iyz = "0"
               izz="${m*(l*l+b*b)/12}" />
-  </macro>
-  <macro name="sphere_inertia" params="m r">
+  </xacro:macro>
+  <xacro:macro name="sphere_inertia" params="m r">
     <inertia  ixx="${2*m*(r*r)/3}" ixy = "0" ixz = "0"
               iyy="${2*m*(r*r)/3}" iyz = "0"
               izz="${2*m*(r*r)/3}" />
-  </macro>
+  </xacro:macro>
   <!-- Wheels -->
-  <property name="wheel_radius" value="0.05" />
-  <property name="wheel_height" value="0.045" />
-  <property name="wheel_mass" value="0.2" />
-  <property name="base_x_origin_to_wheel_origin" value="0.16" />
-  <property name="base_y_origin_to_wheel_origin" value="0.1055" />
-  <property name="base_z_origin_to_wheel_origin" value="0" />
-  <property name="base_x_sphere_origin_to_wheel_origin" value="0.000" />
-  <property name="base_y_sphere_origin_to_wheel_origin" value="0.001" />
-  <property name="base_z_sphere_origin_to_wheel_origin" value="0" />
+  <xacro:property name="wheel_radius" value="0.05" />
+  <xacro:property name="wheel_height" value="0.045" />
+  <xacro:property name="wheel_mass" value="0.2" />
+  <xacro:property name="base_x_origin_to_wheel_origin" value="0.16" />
+  <xacro:property name="base_y_origin_to_wheel_origin" value="0.1055" />
+  <xacro:property name="base_z_origin_to_wheel_origin" value="0" />
+  <xacro:property name="base_x_sphere_origin_to_wheel_origin" value="0.000" />
+  <xacro:property name="base_y_sphere_origin_to_wheel_origin" value="0.001" />
+  <xacro:property name="base_z_sphere_origin_to_wheel_origin" value="0" />
   <xacro:macro name="wheel" params="fb lr parent translateX translateY left OffsetJointX OffsetJointY OffsetJointZ OffsetY">
     <link name="${lr}_wheel_${fb}">
@@ -71,6 +71,6 @@
   </xacro:macro>
   <!-- Steering -->
-  <property name="steering_radius" value="0.01" />
-  <property name="steering_mass" value="0.07" />
+  <xacro:property name="steering_radius" value="0.01" />
+  <xacro:property name="steering_mass" value="0.07" />
   <xacro:macro name="steering_hinge" params="lr parent translateY OffsetY">
     <link name="${lr}_steering">
